Commit message: update ur_automata_moveit_config

File: src/automata_robot/ur_automata_description/urdf/ur_automata.urdf.xacro (robot description, xacro)
@@ -1,26 +1,98 @@
 <?xml version="1.0"?>
 <robot xmlns:xacro="http://wiki.ros.org/xacro" name="ur_automata">
-  <xacro:arg name="name" default="ur"/>
+  <xacro:arg name="name" default="ur_automata"/>
+  <xacro:include filename="$(find ur_description)/urdf/ur_macro.xacro"/>
+  <xacro:include filename="$(find ur_robot_driver)/urdf/ur.ros2_control.xacro" />
+  <xacro:include filename="$(find ur_description)/urdf/inc/ur_transmissions.xacro" />
   <xacro:arg name="ur_type" default="ur5e"/>
-  <link name="world"/>
-  <xacro:include filename="$(find ur_description)/urdf/ur_macro.xacro"/>
+  <xacro:arg name="tf_prefix" default="" />
+  <xacro:arg name="joint_limit_params" default="$(find ur_description)/config/$(arg ur_type)/joint_limits.yaml"/>
+  <xacro:arg name="kinematics_params" default="$(find ur_description)/config/$(arg ur_type)/default_kinematics.yaml"/>
+  <xacro:arg name="physical_params" default="$(find ur_description)/config/$(arg ur_type)/physical_parameters.yaml"/>
+  <xacro:arg name="visual_params" default="$(find ur_description)/config/$(arg ur_type)/visual_parameters.yaml"/>
+  <xacro:arg name="transmission_hw_interface" default=""/>
+  <xacro:arg name="safety_limits" default="false"/>
+  <xacro:arg name="safety_pos_margin" default="0.15"/>
+  <xacro:arg name="safety_k_position" default="20"/>
+  <xacro:arg name="headless_mode" default="false" />
+  <xacro:arg name="robot_ip" default="0.0.0.0" />
+  <xacro:arg name="script_filename" default=""/>
+  <xacro:arg name="output_recipe_filename" default=""/>
+  <xacro:arg name="input_recipe_filename" default=""/>
+  <xacro:arg name="reverse_ip" default="0.0.0.0"/>
+  <xacro:arg name="script_command_port" default="50004"/>
+  <xacro:arg name="reverse_port" default="50001"/>
+  <xacro:arg name="script_sender_port" default="50002"/>
+  <xacro:arg name="trajectory_port" default="50003"/>
+  <xacro:arg name="use_tool_communication" default="false" />
+  <xacro:arg name="tool_voltage" default="0" />
+  <xacro:arg name="tool_parity" default="0" />
+  <xacro:arg name="tool_baud_rate" default="115200" />
+  <xacro:arg name="tool_stop_bits" default="1" />
+  <xacro:arg name="tool_rx_idle_chars" default="1.5" />
+  <xacro:arg name="tool_tx_idle_chars" default="3.5" />
+  <xacro:arg name="tool_device_name" default="/tmp/ttyUR" />
+  <xacro:arg name="tool_tcp_port" default="54321" />
+  <xacro:arg name="use_mock_hardware" default="false" />
+  <xacro:arg name="mock_sensor_commands" default="false" />
+  <xacro:arg name="simulation_controllers" default="" />
+  <xacro:arg name="initial_positions_file" default="$(find ur_description)/config/initial_positions.yaml"/>
+  <xacro:property name="initial_positions_file_prop" value="$(arg initial_positions_file)"/>
+  <link name="world" />
   <xacro:ur_robot
     name="$(arg name)"
-    tf_prefix=""
+    tf_prefix="$(arg tf_prefix)"
     parent="world"
-    joint_limits_parameters_file="$(find ur_description)/config/$(arg ur_type)/joint_limits.yaml"
-    kinematics_parameters_file="$(find ur_description)/config/$(arg ur_type)/default_kinematics.yaml"
-    physical_parameters_file="$(find ur_description)/config/$(arg ur_type)/physical_parameters.yaml"
-    visual_parameters_file="$(find ur_description)/config/$(arg ur_type)/visual_parameters.yaml">
+    joint_limits_parameters_file="$(arg joint_limit_params)"
+    kinematics_parameters_file="$(arg kinematics_params)"
+    physical_parameters_file="$(arg physical_params)"
+    visual_parameters_file="$(arg visual_params)"
+    safety_limits="$(arg safety_limits)"
+    safety_pos_margin="$(arg safety_pos_margin)"
+    safety_k_position="$(arg safety_k_position)"
+    >
+     <origin xyz="0 0 0" rpy="0 0 0" />
+  </xacro:ur_robot>
+  <xacro:ur_ros2_control
+    name="$(arg name)"
+    tf_prefix="$(arg tf_prefix)"
+    kinematics_parameters_file="$(arg kinematics_params)"
+    transmission_hw_interface="$(arg transmission_hw_interface)"
+    use_mock_hardware="$(arg use_mock_hardware)"
+    mock_sensor_commands="$(arg mock_sensor_commands)"
+    headless_mode="$(arg headless_mode)"
+    initial_positions="${xacro.load_yaml(initial_positions_file_prop)}"
+    use_tool_communication="$(arg use_tool_communication)"
+    tool_voltage="$(arg tool_voltage)"
+    tool_parity="$(arg tool_parity)"
+    tool_baud_rate="$(arg tool_baud_rate)"
+    tool_stop_bits="$(arg tool_stop_bits)"
+    tool_rx_idle_chars="$(arg tool_rx_idle_chars)"
+    tool_tx_idle_chars="$(arg tool_tx_idle_chars)"
+    tool_device_name="$(arg tool_device_name)"
+    tool_tcp_port="$(arg tool_tcp_port)"
+    robot_ip="$(arg robot_ip)"
+    script_filename="$(arg script_filename)"
+    output_recipe_filename="$(arg output_recipe_filename)"
+    input_recipe_filename="$(arg input_recipe_filename)"
+    reverse_ip="$(arg reverse_ip)"
+    script_command_port="$(arg script_command_port)"
+    reverse_port="$(arg reverse_port)"
+    script_sender_port="$(arg script_sender_port)"
+    trajectory_port="$(arg trajectory_port)"
+  />
+  <joint name="ee_automata_mesh_fixed_joint" type="fixed">
     <origin xyz="0 0 0" rpy="0 0 0"/>
-  </xacro:ur_robot>
+    <parent link="tool0"/>
+    <child link="ee_automata_mesh_link"/>
+  </joint>
   <link name="ee_automata_mesh_link">
     <visual>
       <origin xyz="0 0 0" rpy="0 0 0"/>
       <geometry>
-        <mesh filename="package://ur_automata_description/meshes/ee_automata_01_nogr.stl" scale="0.001 0.001 0.001"/>
+        <mesh filename="package://ur_automata_description/meshes/ee_automata_V1.stl" scale="0.001 0.001 0.001"/>
       </geometry>
-      <material name="slate_grey">
-        <color rgba="0.44 0.50 0.56 1.0"/>
+      <material name="charcoal_grey">
+        <color rgba="0.13 0.13 0.13 1.0"/>
       </material>
     </visual>
@@ -28,18 +100,13 @@
       <origin xyz="0 0 0" rpy="0 0 0"/>
       <geometry>
-        <mesh filename="package://ur_automata_description/meshes/ee_automata_01_nogr.stl" scale="0.001 0.001 0.001"/>
+        <mesh filename="package://ur_automata_description/meshes/ee_automata_V1.stl" scale="0.001 0.001 0.001"/>
       </geometry>
     </collision>
   </link>
-  <joint name="ee_automata_mesh_fixed_joint" type="fixed">
+  <joint name="ee_automata_fixed_joint" type="fixed">
+    <origin xyz="0 0.052 0.153" rpy="0 0 0"/>
     <parent link="tool0"/>
-    <child link="ee_automata_mesh_link"/>
-    <origin xyz="0 0 0" rpy="0 0 0"/>
+    <child link="ee_automata_tcp"/>
   </joint>
-  <link name="ee_automata_link"/>
-  <joint name="ee_automata_fixed_joint" type="fixed">
-    <parent link="tool0"/>
-    <child link="ee_automata_link"/>
-    <origin xyz="0 0.052 0.153" rpy="0 0 0"/>
-  </joint>
+  <link name="ee_automata_tcp"/>
 </robot>

Commit message: add ur_automata_scan pkg

File: src/automata_robot/ur_automata_description/urdf/ur_automata.urdf.xacro (robot description, xacro)
@@ -93,6 +93,6 @@
         <mesh filename="package://ur_automata_description/meshes/ee_automata_V1.stl" scale="0.001 0.001 0.001"/>
       </geometry>
-      <material name="charcoal_grey">
-        <color rgba="0.13 0.13 0.13 1.0"/>
+      <material name="aluminum">
+        <color rgba="0.78 0.78 0.80 1.0"/>
       </material>
     </visual>
