Commit message: Switch scene platform to disk mesh, use EE V2 and URSim config
- scene: platform.stl -> disk.stl (kept platform00/platform01 as alternatives), platform y 0.60 -> 0.50
- urdf: end effector mesh ee_automata_V1 -> ee_automata_V2
- config: robot.ip set to URSim (192.168.56.101), scan center y 0.40 -> 0.30

File: src/automata_robot/ur_automata_description/urdf/ur_automata.urdf.xacro (robot description, xacro)
@@ -91,5 +91,5 @@
       <origin xyz="0 0 0" rpy="0 0 0"/>
       <geometry>
-        <mesh filename="package://ur_automata_description/meshes/ee_automata_V1.stl" scale="0.001 0.001 0.001"/>
+        <mesh filename="package://ur_automata_description/meshes/ee_automata_V2.stl" scale="0.001 0.001 0.001"/>
       </geometry>
       <material name="aluminum">
@@ -100,5 +100,5 @@
       <origin xyz="0 0 0" rpy="0 0 0"/>
       <geometry>
-        <mesh filename="package://ur_automata_description/meshes/ee_automata_V1.stl" scale="0.001 0.001 0.001"/>
+        <mesh filename="package://ur_automata_description/meshes/ee_automata_V2.stl" scale="0.001 0.001 0.001"/>
       </geometry>
     </collision>

Commit message: Make the robot base pose configurable from automata_config.yaml
New keys robot.base_xyz / robot.base_rpy (metres, radians, world frame).
The xacro reads them with xacro.load_yaml and puts them in the origin of
the world -> base_link joint, so the driver and MoveIt build the same URDF
without extra launch arguments; missing keys mean base at the origin.

Meant for trying alternative mountings in simulation, e.g. the robot on a
wall at platform height with the pan axis pointing at the scan sphere:
xyz [0.133, -0.25, 0.455], rpy [-1.5708, 0, 0].

File: src/automata_robot/ur_automata_description/urdf/ur_automata.urdf.xacro (robot description, xacro)
@@ -39,4 +39,11 @@
   <xacro:arg name="initial_positions_file" default="$(find ur_automata_moveit_config)/config/initial_positions.yaml"/>
   <xacro:property name="initial_positions_file_prop" value="$(arg initial_positions_file)"/>
+  <!-- Posa della base nel mondo, letta da automata_config.yaml (robot.base_xyz /
+       base_rpy): driver e MoveIt generano la stessa URDF senza argomenti extra ai
+       launch. Chiavi assenti = base in origine. -->
+  <xacro:property name="automata_config_file" value="$(find ur_automata_bringup)/config/automata_config.yaml"/>
+  <xacro:property name="automata_config" value="${xacro.load_yaml(automata_config_file)}"/>
+  <xacro:property name="base_xyz" value="${automata_config['robot'].get('base_xyz', [0, 0, 0])}"/>
+  <xacro:property name="base_rpy" value="${automata_config['robot'].get('base_rpy', [0, 0, 0])}"/>
   <link name="world" />
   <xacro:ur_robot
@@ -52,5 +59,5 @@
     safety_k_position="$(arg safety_k_position)"
     >
-     <origin xyz="0 0 0" rpy="0 0 0" />
+     <origin xyz="${base_xyz[0]} ${base_xyz[1]} ${base_xyz[2]}" rpy="${base_rpy[0]} ${base_rpy[1]} ${base_rpy[2]}" />
   </xacro:ur_robot>
   <xacro:ur_ros2_control

Commit message: Description: put the TCP on the lens center of the V2 end effector
The TCP offset (0, 0.052, 0.153) was set for the V1 end effector. On
ee_automata_V2.stl the lens rings (same sizes as V1) are centered at
x 0, z 174.5 mm, with the lens barrel axis along Y (the viewing
direction) and the front face still at y 52 mm: the camera sat 21.5 mm
above the point the scan was planned for.

File: src/automata_robot/ur_automata_description/urdf/ur_automata.urdf.xacro (robot description, xacro)
@@ -111,6 +111,9 @@
     </collision>
   </link>
+  <!-- Camera optical center on ee_automata_V2.stl: lens rings centered at
+       x 0, z 174.5 mm (lens barrel axis parallel to Y, the viewing direction),
+       front face at y 52 mm. V1 had the lens at z 153. -->
   <joint name="ee_automata_fixed_joint" type="fixed">
-    <origin xyz="0 0.052 0.153" rpy="0 0 0"/>
+    <origin xyz="0 0.052 0.1745" rpy="0 0 0"/>
     <parent link="tool0"/>
     <child link="ee_automata_tcp"/>
